Commit message: MyzharBot-v4 description almost complete

File: myzharbot_description/urdf/active_sprocket.urdf.xacro (robot description, xacro)
@@ -7,5 +7,5 @@
           <cylinder length="${active_sprocket_leght}" radius="${active_sprocket_radius}"/>
         </geometry>
-        <material name="DarkGrey" />
+        <material name="White" />
       </visual>
       <collision>

File: myzharbot_description/urdf/myzharbot.urdf.xacro (robot description, xacro)
@@ -6,5 +6,5 @@
   <xacro:include filename="$(find myzharbot_description)/urdf/active_sprocket.urdf.xacro" />
   <xacro:include filename="$(find myzharbot_description)/urdf/motor.urdf.xacro" />
-  <xacro:include filename="$(find myzharbot_description)/urdf/sensors/asus_xtion_pro.urdf.xacro"/>
+  <xacro:include filename="$(find myzharbot_description)/urdf/sensors/zed.urdf.xacro"/>
   <!-- Included URDF/XACRO Files -->
   <!-- Global properties -->
@@ -12,23 +12,28 @@
   <!-- Global properties -->
   <!-- Sprockets params -->
-  <property name="active_sprocket_radius" value="0.047625"/>
-  <property name="passive_sprocket_radius" value="0.047625"/>
-  <property name="active_sprocket_leght" value="0.034925"/>
+  <property name="passive_sprocket_radius" value="0.06"/>
   <property name="passive_sprocket_leght" value="0.008"/>
-  <property name="passive_sprocket_offset_x" value="0.135"/>
-  <property name="passive_sprocket_offset_y" value="0.165"/>
-  <property name="passive_sprocket_offset_z" value="0.047625"/>
-  <property name="active_sprocket_offset_x" value="-0.055"/>
-  <property name="active_sprocket_offset_y" value="0.165"/>
-  <property name="active_sprocket_offset_z" value="0.150"/>
+  <property name="passive_sprocket_offset_x" value="0.1749"/>
+  <property name="passive_sprocket_offset_y" value="0.170"/>
+  <property name="passive_sprocket_offset_z" value="0.06"/>
+  <property name="active_sprocket_radius" value="0.06"/>
+  <property name="active_sprocket_leght" value="0.05"/>
+  <property name="active_sprocket_offset_x" value="-0.09663"/>
+  <property name="active_sprocket_offset_y" value="0.170"/>
+  <property name="active_sprocket_offset_z" value="0.140"/>
   <!-- Sprockets params -->
-  <!-- Asus Xtion params -->
+  <!-- Body params -->
+  <property name="base_tickness" value="0.005"/>
+  <property name="main_body_height" value="0.15"/>
+  <property name="jetson_chassis_height" value="0.05"/>
+  <!-- Body params -->
+  <!-- ZED params -->
   <property name="cam_px" value="0.095" />
-  <property name="cam_py" value="0.022" />
-  <property name="cam_pz" value="0.1825" />
+  <property name="cam_py" value="0.06" />
+  <property name="cam_pz" value="0.245" />
   <property name="cam_or" value="0" />
   <property name="cam_op" value="0" />
   <property name="cam_oy" value="0" />
-  <!-- Asus Xtion params -->
+  <!-- ZED params -->
   <!-- base_link -->
   <link name="base_link">
@@ -46,7 +51,7 @@
     <visual>
       <geometry>
-        <box size="0.27 0.27 .005"/>
+        <box size="0.336 0.285 ${base_tickness}"/>
       </geometry>
-      <material name="Black" />
+      <material name="White" />
     </visual>
   </link>
@@ -55,5 +60,5 @@
     <parent link="base_link"/>
     <child link="body_bottom_chassis_link"/>
-    <origin rpy="0 0 0" xyz="0 0 ${passive_sprocket_offset_z+0.01}"/>
+    <origin rpy="0 0 0" xyz="-0.0085 0 ${passive_sprocket_offset_z+base_tickness/2}"/>
     <joint_properties damping="0.0" friction="0.0"/>
   </joint>
@@ -61,7 +66,7 @@
     <visual>
       <geometry>
-        <box size="0.27 0.17 .055"/>
+        <box size="0.336 0.235 ${main_body_height}"/>
       </geometry>
-      <material name="Black" />
+      <material name="White" />
     </visual>
   </link>
@@ -70,19 +75,19 @@
     <parent link="base_link"/>
     <child link="body_top_chassis_link"/>
-    <origin rpy="0 0 0" xyz="0 0 ${passive_sprocket_offset_z+0.0375}"/>
+    <origin rpy="0 0 0" xyz="-0.0085 0 ${passive_sprocket_offset_z+main_body_height/2+base_tickness}"/>
     <joint_properties damping="0.0" friction="0.0"/>
   </joint>
-  <link name="asus_support_link">
+  <link name="zed_support_link">
     <visual>
       <geometry>
         <box size="0.015 0.015 .015"/>
       </geometry>
-      <material name="Black" />
+      <material name="White" />
     </visual>
   </link>
-  <joint name="Asus_support" type="fixed">
+  <joint name="Zed_support" type="fixed">
     <axis xyz="0 0 1"/>
     <parent link="base_link"/>
-    <child link="asus_support_link"/>
+    <child link="zed_support_link"/>
     <origin rpy="0 0 0" xyz="${cam_px-0.01725} 0 0.1575"/>
     <joint_properties damping="0.0" friction="0.0"/>
@@ -93,7 +98,7 @@
     <visual>
       <geometry>
-        <box size="0.13 0.15 .095"/>
+        <box size="0.27 0.27 ${jetson_chassis_height}"/>
       </geometry>
-      <material name="Black" />
+      <material name="White" />
     </visual>
   </link>
@@ -102,11 +107,11 @@
     <parent link="base_link"/>
     <child link="jetson_chassis_link"/>
-    <origin rpy="0 0 0" xyz="0.035 0 ${passive_sprocket_offset_z+0.0125+0.0475}"/>
+    <origin rpy="0 0 0" xyz="-0.04 0 ${passive_sprocket_offset_z+main_body_height+base_tickness+jetson_chassis_height/2}"/>
     <joint_properties damping="0.0" friction="0.0"/>
   </joint>
   <!-- Jetson chassis -->
-  <!-- Asus Xtion Pro Live -->
-  <xacro:sensor_asus_xtion_pro parent="base_link"/>
-  <!-- Asus Xtion Pro Live -->
+  <!-- Stereolabs ZED -->
+  <xacro:sensor_stereolabs_zed parent="base_link"/>
+  <!-- Stereolabs ZED -->
   <!-- Active Sprockets -->
   <xacro:myzharbot_active_sprocket position="Left">
@@ -117,8 +122,8 @@
   </xacro:myzharbot_active_sprocket>
   <xacro:myzharbot_motor position="Left">
-    <origin xyz="${active_sprocket_offset_x} ${active_sprocket_offset_y-2*active_sprocket_leght} ${active_sprocket_offset_z}" rpy="${-M_PI/2} 0 0" />
+    <origin xyz="${active_sprocket_offset_x} ${active_sprocket_offset_y-active_sprocket_leght/2} ${active_sprocket_offset_z}" rpy="${-M_PI/2} 0 0" />
   </xacro:myzharbot_motor>
   <xacro:myzharbot_motor position="Right">
-    <origin xyz="${active_sprocket_offset_x} ${-(active_sprocket_offset_y-2*active_sprocket_leght)} ${active_sprocket_offset_z}" rpy="${-M_PI/2} 0 0" />
+    <origin xyz="${active_sprocket_offset_x} ${-(active_sprocket_offset_y-active_sprocket_leght/2)} ${active_sprocket_offset_z}" rpy="${-M_PI/2} 0 0" />
   </xacro:myzharbot_motor>
   <!-- Active Sprockets -->

File: myzharbot_description/urdf/passive_sprocket.urdf.xacro (robot description, xacro)
@@ -7,5 +7,5 @@
           <cylinder length="${passive_sprocket_leght}" radius="${passive_sprocket_radius}"/>
         </geometry>
-        <material name="DarkGrey" />
+        <material name="White" />
       </visual>
     </link>

Commit message: Added ZED model and launch file  * modified MyzharBot description

File: myzharbot_description/urdf/active_sprocket.urdf.xacro (robot description, xacro)
@@ -7,5 +7,5 @@
           <cylinder length="${active_sprocket_leght}" radius="${active_sprocket_radius}"/>
         </geometry>
-        <material name="White" />
+        <material name="LightGreyT" />
       </visual>
       <collision>

File: myzharbot_description/urdf/myzharbot.urdf.xacro (robot description, xacro)
@@ -29,7 +29,7 @@
   <!-- Body params -->
   <!-- ZED params -->
-  <property name="cam_px" value="0.095" />
+  <property name="cam_px" value="0.0725" />
   <property name="cam_py" value="0.06" />
-  <property name="cam_pz" value="0.245" />
+  <property name="cam_pz" value="0.238" />
   <property name="cam_or" value="0" />
   <property name="cam_op" value="0" />
@@ -53,5 +53,5 @@
         <box size="0.336 0.285 ${base_tickness}"/>
       </geometry>
-      <material name="White" />
+      <material name="LightGreyT" />
     </visual>
   </link>
@@ -68,5 +68,5 @@
         <box size="0.336 0.235 ${main_body_height}"/>
       </geometry>
-      <material name="White" />
+      <material name="LightGreyT" />
     </visual>
   </link>
@@ -78,19 +78,4 @@
     <joint_properties damping="0.0" friction="0.0"/>
   </joint>
-  <link name="zed_support_link">
-    <visual>
-      <geometry>
-        <box size="0.015 0.015 .015"/>
-      </geometry>
-      <material name="White" />
-    </visual>
-  </link>
-  <joint name="Zed_support" type="fixed">
-    <axis xyz="0 0 1"/>
-    <parent link="base_link"/>
-    <child link="zed_support_link"/>
-    <origin rpy="0 0 0" xyz="${cam_px-0.01725} 0 0.1575"/>
-    <joint_properties damping="0.0" friction="0.0"/>
-  </joint>
   <!-- Body chassis -->
   <!-- Jetson chassis -->
@@ -100,5 +85,5 @@
         <box size="0.27 0.27 ${jetson_chassis_height}"/>
       </geometry>
-      <material name="White" />
+      <material name="LightGreyT" />
     </visual>
   </link>

File: myzharbot_description/urdf/passive_sprocket.urdf.xacro (robot description, xacro)
@@ -7,5 +7,5 @@
           <cylinder length="${passive_sprocket_leght}" radius="${passive_sprocket_radius}"/>
         </geometry>
-        <material name="White" />
+        <material name="LightGreyT" />
       </visual>
     </link>

File: myzharbot_description/urdf/sensors/asus_xtion_pro.urdf.xacro (robot description, xacro)
@@ -32,4 +32,5 @@
           <mesh filename="package://ros_myzharbot_robot/meshes/sensors/asus_xtion_pro_live.dae" scale="${M_SCALE} ${M_SCALE} ${M_SCALE}"/>
         </geometry>
+        <material name="DarkGrey" />
       </visual>
       <collision>

File: myzharbot_description/urdf/sensors/zed.urdf.xacro (robot description, xacro)
@@ -1,4 +1,5 @@
 <?xml version="1.0"?>
 <robot name="sensor_stereolabs_zed" xmlns:xacro="http://ros.org/wiki/xacro">
+  <!-- Included URDF/XACRO Files -->
   <!-- Xacro properties -->
   <xacro:property name="M_SCALE" value="0.001"/>
@@ -6,29 +7,30 @@
   <!-- Parameterised in part by the values in turtlebot_properties.urdf.xacro -->
   <xacro:macro name="sensor_stereolabs_zed" params="parent">
-    <joint name="stereo_camera_left_joint" type="fixed">
+    <joint name="zed_left_joint" type="fixed">
       <origin xyz="${cam_px} ${cam_py} ${cam_pz}"
               rpy="${cam_or} ${cam_op} ${cam_oy}"/>
       <parent link="${parent}"/>
-      <child link="stereo_camera_left_frame" />
+      <child link="zed_left_frame" />
     </joint>
-    <link name="stereo_camera_left_frame"/>
-    <joint name="camera_left_optical_joint" type="fixed">
+    <link name="zed_left_frame"/>
+    <joint name="zed_left_optical_joint" type="fixed">
       <origin xyz="0 0 0" rpy="${-M_PI/2} 0 ${-M_PI/2}" />
-      <parent link="stereo_camera_left_frame" />
-      <child link="stereo_camera_left_optical_frame" />
+      <parent link="zed_left_frame" />
+      <child link="zed_left_optical_frame" />
     </joint>
-    <link name="stereo_camera_left_optical_frame"/>
+    <link name="zed_left_optical_frame"/>
     <joint name="_camera_joint" type="fixed">
       <origin xyz="0 ${-optical_y_offset} 0"
               rpy="0 0 0"/>
-      <parent link="stereo_camera_left_frame"/>
-      <child link="stereo_camera_link"/>
+      <parent link="zed_left_frame"/>
+      <child link="zed_camera_link"/>
     </joint>
-    <link name="stereo_camera_link">
+    <link name="zed_camera_link">
       <visual>
         <origin xyz="-0.01 0 0" rpy="${-M_PI/2} -${M_PI} ${-M_PI/2}"/>
         <geometry>
-          <mesh filename="package://myzharbot_description/meshes/sensors/asus_xtion_pro_live.dae" scale="${M_SCALE} ${M_SCALE} ${M_SCALE}"/>
+          <mesh filename="package://myzharbot_description/meshes/sensors/stereolabs_zed.STL" scale="${M_SCALE} ${M_SCALE} ${M_SCALE}"/>
         </geometry>
+        <material name="DarkGrey" />
       </visual>
       <collision>
@@ -46,16 +48,16 @@
       </inertial>
     </link>
-    <joint name="stereo_camera_right_joint" type="fixed">
+    <joint name="zed_right_joint" type="fixed">
       <origin xyz="0 ${-2*optical_y_offset} 0" rpy="0 0 0" />
-      <parent link="stereo_camera_left_frame" />
-      <child link="stereo_camera_right_frame" />
+      <parent link="zed_left_frame" />
+      <child link="zed_right_frame" />
     </joint>
-    <link name="stereo_camera_right_frame"/>
-    <joint name="camera_right_optical_joint" type="fixed">
+    <link name="zed_right_frame"/>
+    <joint name="zed_right_optical_joint" type="fixed">
       <origin xyz="0 0 0" rpy="${-M_PI/2} 0 ${-M_PI/2}" />
-      <parent link="stereo_camera_right_frame" />
-      <child link="stereo_camera_right_optical_frame" />
+      <parent link="zed_right_frame" />
+      <child link="zed_right_optical_frame" />
     </joint>
-    <link name="stereo_camera_right_optical_frame"/>
+    <link name="zed_right_optical_frame"/>
   </xacro:macro>
 </robot>
