Commit message: First little modifications to Robot Description for MyzharBot-v4

File: myzharbot_description/urdf/myzharbot.urdf.xacro (robot description, xacro)
@@ -1,4 +1,4 @@
 <?xml version="1.0"?>
-<robot name="myzharbot_robot" xmlns:xacro="http://ros.org/wiki/xacro">
+<robot name="myzharbot" xmlns:xacro="http://ros.org/wiki/xacro">
   <!-- Included URDF/XACRO Files -->
   <xacro:include filename="$(find myzharbot_description)/urdf/materials.urdf" />
@@ -15,10 +15,10 @@
   <property name="passive_sprocket_radius" value="0.047625"/>
   <property name="active_sprocket_leght" value="0.034925"/>
-  <property name="passive_sprocket_leght" value="0.047625"/>
+  <property name="passive_sprocket_leght" value="0.008"/>
   <property name="passive_sprocket_offset_x" value="0.135"/>
   <property name="passive_sprocket_offset_y" value="0.165"/>
   <property name="passive_sprocket_offset_z" value="0.047625"/>
   <property name="active_sprocket_offset_x" value="-0.055"/>
-  <property name="active_sprocket_offset_y" value="0.160"/>
+  <property name="active_sprocket_offset_y" value="0.165"/>
   <property name="active_sprocket_offset_z" value="0.150"/>
   <!-- Sprockets params -->
@@ -61,5 +61,5 @@
     <visual>
       <geometry>
-        <box size="0.13 0.27 .055"/>
+        <box size="0.27 0.17 .055"/>
       </geometry>
       <material name="Black" />
@@ -70,5 +70,5 @@
     <parent link="base_link"/>
     <child link="body_top_chassis_link"/>
-    <origin rpy="0 0 0" xyz="-0.035 0 ${passive_sprocket_offset_z+0.0375}"/>
+    <origin rpy="0 0 0" xyz="0 0 ${passive_sprocket_offset_z+0.0375}"/>
     <joint_properties damping="0.0" friction="0.0"/>
   </joint>

Commit message: Little measure correction

File: myzharbot_description/urdf/myzharbot.urdf.xacro (robot description, xacro)
@@ -25,5 +25,5 @@
   <!-- Body params -->
   <property name="base_tickness" value="0.005"/>
-  <property name="main_body_height" value="0.15"/>
+  <property name="main_body_height" value="0.12"/>
   <property name="jetson_chassis_height" value="0.05"/>
   <!-- Body params -->
@@ -31,5 +31,5 @@
   <property name="cam_px" value="0.0725" />
   <property name="cam_py" value="0.06" />
-  <property name="cam_pz" value="0.238" />
+  <property name="cam_pz" value="0.208" />
   <property name="cam_or" value="0" />
   <property name="cam_op" value="0" />
@@ -107,8 +107,8 @@
   </xacro:myzharbot_active_sprocket>
   <xacro:myzharbot_motor position="Left">
-    <origin xyz="${active_sprocket_offset_x} ${active_sprocket_offset_y-active_sprocket_leght/2} ${active_sprocket_offset_z}" rpy="${-M_PI/2} 0 0" />
+    <origin xyz="${active_sprocket_offset_x} ${active_sprocket_offset_y-0.07} ${active_sprocket_offset_z}" rpy="${-M_PI/2} 0 0" />
   </xacro:myzharbot_motor>
   <xacro:myzharbot_motor position="Right">
-    <origin xyz="${active_sprocket_offset_x} ${-(active_sprocket_offset_y-active_sprocket_leght/2)} ${active_sprocket_offset_z}" rpy="${-M_PI/2} 0 0" />
+    <origin xyz="${active_sprocket_offset_x} ${-(active_sprocket_offset_y-0.07)} ${active_sprocket_offset_z}" rpy="${-M_PI/2} 0 0" />
   </xacro:myzharbot_motor>
   <!-- Active Sprockets -->

Commit message: bug fixes

File: myzharbot_description/urdf/myzharbot.urdf.xacro (robot description, xacro)
@@ -29,10 +29,10 @@
   <!-- Body params -->
   <!-- ZED params -->
-  <property name="cam_px" value="0.0725" />
-  <property name="cam_py" value="0.06" />
-  <property name="cam_pz" value="0.208" />
-  <property name="cam_or" value="0" />
-  <property name="cam_op" value="0" />
-  <property name="cam_oy" value="0" />
+  <property name="zed_px" value="0.0725" />
+  <property name="zed_py" value="0.0" />
+  <property name="zed_pz" value="0.208" />
+  <property name="zed_or" value="0" />
+  <property name="zed_op" value="0" />
+  <property name="zed_oy" value="0" />
   <!-- ZED params -->
   <!-- base_link -->

File: myzharbot_description/urdf/sensors/zed.urdf.xacro (robot description, xacro)
@@ -8,7 +8,7 @@
   <xacro:macro name="sensor_stereolabs_zed" params="parent">
     <joint name="zed_left_joint" type="fixed">
-      <origin xyz="${cam_px} ${cam_py} ${cam_pz}"
-              rpy="${cam_or} ${cam_op} ${cam_oy}"/>
-      <parent link="${parent}"/>
+      <origin xyz="0 ${optical_y_offset} 0"
+              rpy="0 0 0"/>
+      <parent link="zed_camera_link"/>
       <child link="zed_left_frame" />
     </joint>
@@ -21,7 +21,7 @@
     <link name="zed_left_optical_frame"/>
     <joint name="_camera_joint" type="fixed">
-      <origin xyz="0 ${-optical_y_offset} 0"
-              rpy="0 0 0"/>
-      <parent link="zed_left_frame"/>
+      <origin xyz="${zed_px} ${zed_py} ${zed_pz}"
+              rpy="${zed_or} ${zed_op} ${zed_oy}"/>
+      <parent link="${parent}"/>
       <child link="zed_camera_link"/>
     </joint>
@@ -49,6 +49,6 @@
     </link>
     <joint name="zed_right_joint" type="fixed">
-      <origin xyz="0 ${-2*optical_y_offset} 0" rpy="0 0 0" />
-      <parent link="zed_left_frame" />
+      <origin xyz="0 ${-optical_y_offset} 0" rpy="0 0 0" />
+      <parent link="zed_camera_link" />
       <child link="zed_right_frame" />
     </joint>

Commit message: Update before GTC2016

File: myzharbot_description/urdf/myzharbot.urdf.xacro (robot description, xacro)
@@ -7,4 +7,5 @@
   <xacro:include filename="$(find myzharbot_description)/urdf/motor.urdf.xacro" />
   <xacro:include filename="$(find myzharbot_description)/urdf/sensors/zed.urdf.xacro"/>
+  <xacro:include filename="$(find myzharbot_description)/urdf/sensors/imu.urdf.xacro"/>
   <!-- Included URDF/XACRO Files -->
   <!-- Global properties -->
@@ -96,4 +97,10 @@
   </joint>
   <!-- Jetson chassis -->
+  <!-- IMU -->
+  <xacro:imu name="imu" parent="base_link">
+    <!--<origin xyz="0 0 0.22" rpy="0 0 0" />-->
+    <origin xyz="0.0 0.000 0.22" rpy="0 0 0" />
+  </xacro:imu>
+  <!-- IMU -->
   <!-- Stereolabs ZED -->
   <xacro:sensor_stereolabs_zed parent="base_link"/>
